Commit message: Fix Livox Avia model
Signed-off-by: Emiliano Borghi <emiliano@smartmachine.nz>

File: urdf/livox_avia.xacro (robot description, xacro)
@@ -1,5 +1,4 @@
 <?xml version="1.0"?>
 <robot xmlns:xacro="http://ros.org/wiki/xacro">
-  <xacro:property name="M_PI" value="3.14159"/>
   <xacro:property name="laser_min_range" value="0.1"/>
   <xacro:property name="laser_max_range" value="200.0"/>
@@ -8,23 +7,21 @@
   <xacro:property name="ros_topic" value="scan"/>
   <xacro:property name="samples" value="24000"/>
-  <xacro:property name="downsample" value="1"/>
+  <xacro:property name="publish_pointcloud_type" value="0"/>
   <xacro:property name="csv_file_name" value="package://livox_laser_simulation/scan_mode/avia.csv"/>
   <xacro:include filename="$(find livox_laser_simulation)/urdf/livox_gazebo_sensor.xacro"/>
-  <xacro:macro name="Livox_Avia" params="visualize:=True name:=livox publish_pointcloud_type:=0">
+  <xacro:macro name="Livox_Avia" params="visualize:=True name:=livox publish_pointcloud_type:=0
+                                         ros_topic:=livox/lidar downsample:=1
+                                         noise_mean:=0.0 noise_stddev:=0.01 imu_noise_stddev:=0.00264">
     <link name="${name}_base">
       <xacro:null_inertial/>
       <visual>
-        <origin xyz="0.00 0 0.00" rpy="0 0 0"/>
         <geometry>
-          <mesh filename="package://livox_laser_simulation/meshes/livox_mid40.dae">
-          </mesh>
+          <mesh filename="package://livox_laser_simulation/meshes/livox_mid40.dae"/>
         </geometry>
       </visual>
       <collision>
-          <origin xyz="0 0 0" rpy="0 0 0" />
-          <geometry>
-          <mesh filename="package://livox_laser_simulation/meshes/livox_mid40.dae">
-          </mesh>
-          </geometry>
+        <geometry>
+          <mesh filename="package://livox_laser_simulation/meshes/livox_mid40.dae"/>
+        </geometry>
       </collision>
     </link>
@@ -35,7 +32,14 @@
       <parent link="${name}_base"/>
       <child link="${name}"/>
-      <origin rpy="0 0 0" xyz="0.0 0.0 0.0"/>
     </joint>
-    <xacro:Livox_gazebo_sensor name="${name}" visualize="${visualize}" publish_pointcloud_type="${publish_pointcloud_type}"/>
+    <link name="${name}_imu_link"/>
+    <!-- IMU Coordinates: https://terra-1-g.djicdn.com/65c028cd298f4669a7f0e40e50ba1131/demo/avia/Livox%20AVIA%20User%20Manual_EN.pdf -->
+    <joint name="imu_link_joint" type="fixed">
+      <parent link="${name}"/>
+      <child link="${name}_imu_link"/>
+      <origin xyz="-0.04165 -0.02326 0.0284"/>
+    </joint>
+    <xacro:Livox_gazebo_sensor name="${name}" visualize="${visualize}" publish_pointcloud_type="${publish_pointcloud_type}"
+                               noise_mean="${noise_mean}" noise_stddev="${noise_stddev}" imu_noise_stddev="${imu_noise_stddev}"/>
   </xacro:macro>
 </robot>

File: urdf/livox_horizon.xacro (robot description, xacro)
@@ -1,5 +1,4 @@
 <?xml version="1.0"?>
 <robot xmlns:xacro="http://ros.org/wiki/xacro">
-  <xacro:property name="M_PI" value="3.14159"/>
   <xacro:property name="laser_min_range" value="0.1"/>
   <xacro:property name="laser_max_range" value="200.0"/>
@@ -11,20 +10,17 @@
   <xacro:property name="csv_file_name" value="package://livox_laser_simulation/scan_mode/horizon.csv"/>
   <xacro:include filename="$(find livox_laser_simulation)/urdf/livox_gazebo_sensor.xacro"/>
-  <xacro:macro name="Livox_Horizon" params="visualize:=True name:=livox publish_pointcloud_type:=0 ros_topic:=livox/lidar downsample:=1
-                                            noise_mean:=0.0 noise_stddev:=0.01 imu_noise_stddev:=0.0026399240948208127">
+  <xacro:macro name="Livox_Horizon" params="visualize:=True name:=livox publish_pointcloud_type:=0
+                                            ros_topic:=livox/lidar downsample:=1
+                                            noise_mean:=0.0 noise_stddev:=0.01 imu_noise_stddev:=0.00264">
     <link name="${name}_base">
       <xacro:null_inertial/>
       <visual>
-        <origin xyz="0.00 0 0.00" rpy="0 0 0"/>
         <geometry>
-          <mesh filename="package://livox_laser_simulation/meshes/livox_mid40.dae">
-          </mesh>
+          <mesh filename="package://livox_laser_simulation/meshes/livox_mid40.dae"/>
         </geometry>
       </visual>
       <collision>
-		  <origin xyz="0.00 0 0.00" rpy="0 0 0" />
       <geometry>
-        <mesh filename="package://livox_laser_simulation/meshes/livox_mid40.dae">
-		    </mesh>
+        <mesh filename="package://livox_laser_simulation/meshes/livox_mid40.dae"/>
       </geometry>
       </collision>
@@ -36,5 +32,4 @@
       <parent link="${name}_base"/>
       <child link="${name}"/>
-      <origin rpy="0 0 0" xyz="0.0 0.0 0.0"/>
     </joint>
     <link name="${name}_imu_link"/>
@@ -42,5 +37,5 @@
       <parent link="${name}"/>
       <child link="${name}_imu_link"/>
-      <origin rpy="0 0 0" xyz="-0.05512 -0.02226 0.0297"/>
+      <origin xyz="-0.05512 -0.02226 0.0297"/>
     </joint>
     <xacro:Livox_gazebo_sensor name="${name}" visualize="${visualize}" publish_pointcloud_type="${publish_pointcloud_type}"
