Commit message: Don't publish empty cloud
Signed-off-by: Emiliano Borghi <emiliano@smartmachine.nz>

File: urdf/livox_gazebo_sensor.xacro (robot description, xacro)
@@ -4,7 +4,7 @@
     <inertial>
       <mass value="0.1"/>
-    <inertia ixx="0.001" ixy="0" ixz="0"
-          iyy="0.001" iyz="0"
-          izz="0.001"/>
+      <inertia ixx="0.001" ixy="0" ixz="0"
+               iyy="0.001" iyz="0"
+               izz="0.001"/>
     </inertial>
   </xacro:macro>
@@ -51,4 +51,5 @@
           <publish_pointcloud_type>${publish_pointcloud_type}</publish_pointcloud_type>
           <ros_topic>${ros_topic}</ros_topic>
+          <robotNamespace>livox</robotNamespace>
         </plugin>
       </sensor>
@@ -59,5 +60,6 @@
         <visualize>false</visualize>
         <plugin filename="libgazebo_ros_imu_sensor.so" name="imu_plugin">
-          <topicName>/livox/imu</topicName>
+          <robotNamespace>livox</robotNamespace>
+          <topicName>imu</topicName>
           <bodyName>livox_imu_link</bodyName>
           <updateRateHZ>200.0</updateRateHZ>
